Commit message: :

File: ur5e_unity_bridge/urdf/ur5e.urdf (robot description, URDF)
Before this commit: robot ur5e, 13 links, 12 joints
Joints:
- joint shoulder_lift_joint: limit lower=-6.283185307179586 upper=6.283185307179586 effort=150.0 velocity=3.141592653589793 -> lower=-3.14159 upper=3.14159 effort=150.0 velocity=3.14159
- joint shoulder_pan_joint: limit lower=-6.283185307179586 upper=6.283185307179586 effort=150.0 velocity=3.141592653589793 -> lower=-3.14159 upper=3.14159 effort=150.0 velocity=3.14159
- joint wrist_1_joint: limit lower=-6.283185307179586 upper=6.283185307179586 effort=28.0 velocity=3.141592653589793 -> lower=-3.14159 upper=3.14159 effort=28.0 velocity=3.14159
- joint wrist_2_joint: limit lower=-6.283185307179586 upper=6.283185307179586 effort=28.0 velocity=3.141592653589793 -> lower=-3.14159 upper=3.14159 effort=28.0 velocity=3.14159
- joint wrist_3_joint: limit lower=-6.283185307179586 upper=6.283185307179586 effort=28.0 velocity=3.141592653589793 -> lower=-3.14159 upper=3.14159 effort=28.0 velocity=3.14159
